File: CircuitPrincipaleCarbonEye/circuitLedCarbonEye/circuitLedCarbonEye.kicad_pcb (KiCad board)
At the start: 2 copper layers, 40 x 56 mm, 10 parts, among them J1 4P4C

Commit message: KICAD RoutageCircuit led V1.0
Routing:
- net Net-(LED1-Pad2): track 65.6 -> 34.5 mm
- net Net-(J1-Pad2): track 105.0 -> 106.8 mm
- added copper zone on F.Cu, net Net-(LED1-Pad2)

Commit message: mise à jour circuit led pour premiere impresson
Parts:
- added REF**: MountingHole_3.2mm_M3, MountingHole:MountingHole_3.2mm_M3, F.Cu at (240.0, 65.5)
- added REF**: MountingHole_3.2mm_M3, MountingHole:MountingHole_3.2mm_M3, F.Cu at (223.5, 82.0)
- added REF**: MountingHole_3.2mm_M3, MountingHole:MountingHole_3.2mm_M3, F.Cu at (256.5, 82.0)

Commit message: vérification avant impression 1
Parts:
- moved LED2 0.30 mm to (230.3, 82.0)
Routing:
- net Net-(J1-Pad3): track 128.4 -> 112.2 mm
- net Net-(LED1-Pad2): track 34.5 -> 44.9 mm
- net Net-(J1-Pad2): track 106.8 -> 98.4 mm
