File: CircuitPrincipaleCarbonEye/circuitLedCarbonEye/circuitLedCarbonEye.sch (KiCad schematic (older format))
At the start: 10 parts, among them J1 4P4C

Commit message: vérification avant impression 1
Parts:
- LED1, LED2, LED3, LED4, LED5, LED6, LED7, LED8: symbol SamacSys_Parts:VSMG2700-GS08 -> circuitLedCarbonEye-rescue:VSMG2700-GS08-SamacSys_Parts
Changed lines of the file:
@@
 $EndDescr
 $Comp
-L SamacSys_Parts:VSMG2700-GS08 LED4
+L circuitLedCarbonEye-rescue:VSMG2700-GS08-SamacSys_Parts LED4
 U 1 1 60E9C099
 P 4800 2400
@@
 $EndComp
 $Comp
-L SamacSys_Parts:VSMG2700-GS08 LED3
+L circuitLedCarbonEye-rescue:VSMG2700-GS08-SamacSys_Parts LED3
 U 1 1 60E9E6AE
 P 4800 2050
@@
 $EndComp
 $Comp
-L SamacSys_Parts:VSMG2700-GS08 LED2
+L circuitLedCarbonEye-rescue:VSMG2700-GS08-SamacSys_Parts LED2
 U 1 1 60E9F245
 P 4800 1700
@@
 $EndComp
 $Comp
-L SamacSys_Parts:VSMG2700-GS08 LED1
+L circuitLedCarbonEye-rescue:VSMG2700-GS08-SamacSys_Parts LED1
 U 1 1 60E9F8A2
 P 4800 1300
@@
 $EndComp
 $Comp
-L SamacSys_Parts:VSMG2700-GS08 LED5
+L circuitLedCarbonEye-rescue:VSMG2700-GS08-SamacSys_Parts LED5
 U 1 1 60E9FE4B
 P 4800 3150
@@
 $EndComp
 $Comp
-L SamacSys_Parts:VSMG2700-GS08 LED6
+L circuitLedCarbonEye-rescue:VSMG2700-GS08-SamacSys_Parts LED6
 U 1 1 60EA02FE
 P 4800 3500
@@
 $EndComp
 $Comp
-L SamacSys_Parts:VSMG2700-GS08 LED7
+L circuitLedCarbonEye-rescue:VSMG2700-GS08-SamacSys_Parts LED7
 U 1 1 60EA09CD
 P 4800 3850
@@
 $EndComp
 $Comp
-L SamacSys_Parts:VSMG2700-GS08 LED8
+L circuitLedCarbonEye-rescue:VSMG2700-GS08-SamacSys_Parts LED8
 U 1 1 60EA111A
 P 4800 4250
